Commit message: visualisation complete, ready to configure collision plan

File: src/end_effector_description/urdf/end_effector.urdf.xacro (robot description, xacro)
@@ -36,5 +36,5 @@
       <parent link="${parent}"/>
       <child link="${prefix}camera"/>
-      <origin xyz="0 0 0" rpy="${pi/2} 0 0"/>
+      <origin xyz="-0.02 -0.05 -0.135" rpy="${pi/2} 0 0"/>
     </joint>
     <!-- QC link, 5 cm above camera -->
@@ -43,5 +43,5 @@
       <parent link="${prefix}camera"/>
       <child link="${prefix}QC"/>
-      <origin xyz="0.05 0 0" rpy="${pi} 0 0"/>
+      <origin xyz="0.02 0.147 -0.05" rpy="${pi} ${-pi/2} 0"/>
     </joint>
     <!-- Gripper link, 5 cm above QC -->
@@ -50,5 +50,5 @@
       <parent link="${prefix}QC"/>
       <child link="${prefix}gripper"/>
-      <origin xyz="0.15 0 0" rpy="0 ${pi} ${pi/2}"/>
+      <origin xyz="0 -0.067 -0.025" rpy="${-pi/2} ${pi} ${pi/2}"/>
     </joint>
   </xacro:macro>
