Commit message: add custom moveit config package that changes to RRTConnect Planner, no joint constraints needed anymore, need further cleanup

File: src/end_effector_description/urdf/end_effector_withDriverSupport.xacro (robot description, xacro)
@@ -13,5 +13,6 @@
       <parent link="flange"/>
       <child link="camera_link"/>
-      <origin xyz="0.0345 0 -0.1032" rpy="${pi} ${pi} ${pi}"/>
+      <!-- <origin xyz="0.0345 0 -0.1032" rpy="${pi} ${pi} ${pi}"/> -->
+      <origin xyz="0.0199931 -0.0028582 -0.109958" rpy="3.12825 -3.12574 -3.13495" />
   </joint>
 </robot>

Commit message: added stl files, initial setup complete, need to tune positioning next

File: src/end_effector_description/urdf/end_effector_withDriverSupport.xacro (robot description, xacro)
@@ -3,5 +3,5 @@
 <robot name="end_effector_withDriverSupport" xmlns:xacro="http://ros.org/wiki/xacro">
   <!-- Including the claw.urdf.xacro file to give scope to xacro:claw. Inclusion is a simple copy-and-paste of code. -->
-  <!-- <xacro:include filename="$(find end_effector_description)/urdf/end_effector.urdf.xacro" /> -->
+  <xacro:include filename="$(find end_effector_description)/urdf/end_effector.urdf.xacro" />
   <!-- UR5e robot arm -->
   <!-- URDF won't build if following args aren't defined. -->
@@ -9,4 +9,14 @@
   <xacro:arg name="ur_type" default="ur10"/>
   <xacro:include filename="$(find ur_description)/urdf/ur.urdf.xacro"/>
+  <!-- This is the abstract link which the base of the claw attaches to. -->
+  <link name="end_effector_root_link"/>
+  <!-- Instantiate the claw by using its macro. -->
+  <xacro:end_effector prefix="" parent="end_effector_root_link" >
+  </xacro:end_effector>
+  <!-- Coupler between arm and end effector -->
+  <joint name="end_effector_coupler_joint" type="fixed">
+    <parent link="tool0"/>
+    <child link="end_effector_root_link"/>
+  </joint>
   <link name="camera_link"> </link>
   <joint name="camera_joint" type="fixed">

Commit message: at least it is working now, crzy swinging motions and all

File: src/end_effector_description/urdf/end_effector_withDriverSupport.xacro (robot description, xacro)
@@ -9,4 +9,34 @@
   <xacro:arg name="ur_type" default="ur10"/>
   <xacro:include filename="$(find ur_description)/urdf/ur.urdf.xacro"/>
+ <!-- Simple rectangular end-effector -->
+  <link name="simple_ee_link">
+    <visual>
+      <geometry>
+        <box size="0.15 0.15 0.3"/>  <!-- Length, Width, Height -->
+      </geometry>
+      <material name="orange">
+        <color rgba="1.0 0.5 0.0 1.0"/>
+      </material>
+    </visual>
+    <collision>
+      <geometry>
+        <box size="0.15 0.15 0.3"/>  <!-- Must match visual -->
+      </geometry>
+    </collision>
+    <inertial>
+    <mass value="2.0"/>  <!-- 2kg mass -->
+    <!-- Calculated inertia for a rectangular prism -->
+    <inertia
+      ixx="0.01625" ixy="0.0" ixz="0.0"
+      iyy="0.0085" iyz="0.0"
+      izz="0.00425"/>
+  </inertial>
+  </link>
+  <!-- Fixed joint attaching to tool0 -->
+  <joint name="simple_ee_joint" type="fixed">
+    <parent link="tool0"/>
+    <child link="simple_ee_link"/>
+    <origin xyz="0 -0.02 0.16" rpy="0 0 0"/>  <!-- 1cm offset from tool0 -->
+  </joint>
   <link name="camera_link"> </link>
   <joint name="camera_joint" type="fixed">

Commit message: David fix srdf & add motion planning server functionalities (#1)

File: src/end_effector_description/urdf/end_effector_withDriverSupport.xacro (robot description, xacro)
@@ -9,13 +9,33 @@
   <xacro:arg name="ur_type" default="ur10"/>
   <xacro:include filename="$(find ur_description)/urdf/ur.urdf.xacro"/>
-  <!-- This is the abstract link which the base of the claw attaches to. -->
-  <link name="end_effector_root_link"/>
-  <!-- Instantiate the claw by using its macro. -->
-  <xacro:end_effector prefix="" parent="end_effector_root_link" >
-  </xacro:end_effector>
-  <!-- Coupler between arm and end effector -->
-  <joint name="end_effector_coupler_joint" type="fixed">
+ <!-- Simple rectangular end-effector -->
+  <link name="simple_ee_link">
+    <visual>
+      <geometry>
+        <box size="0.15 0.15 0.3"/>  <!-- Length, Width, Height -->
+      </geometry>
+      <material name="orange">
+        <color rgba="1.0 0.5 0.0 1.0"/>
+      </material>
+    </visual>
+    <collision>
+      <geometry>
+        <box size="0.15 0.15 0.3"/>  <!-- Must match visual -->
+      </geometry>
+    </collision>
+    <inertial>
+    <mass value="2.0"/>  <!-- 2kg mass -->
+    <!-- Calculated inertia for a rectangular prism -->
+    <inertia
+      ixx="0.01625" ixy="0.0" ixz="0.0"
+      iyy="0.0085" iyz="0.0"
+      izz="0.00425"/>
+  </inertial>
+  </link>
+  <!-- Fixed joint attaching to tool0 -->
+  <joint name="simple_ee_joint" type="fixed">
     <parent link="tool0"/>
-    <child link="end_effector_root_link"/>
+    <child link="simple_ee_link"/>
+    <origin xyz="0 -0.02 0.16" rpy="0 0 0"/>  <!-- 1cm offset from tool0 -->
   </joint>
   <link name="camera_link"> </link>

Commit message: fix horizontal gripping demo

File: src/end_effector_description/urdf/end_effector_withDriverSupport.xacro (robot description, xacro)
@@ -13,5 +13,5 @@
     <visual>
       <geometry>
-        <box size="0.15 0.15 0.3"/>  <!-- Length, Width, Height -->
+        <box size="0.15 0.15 0.2"/>  <!-- Length, Width, Height -->
       </geometry>
       <material name="orange">
@@ -21,5 +21,5 @@
     <collision>
       <geometry>
-        <box size="0.15 0.15 0.3"/>  <!-- Must match visual -->
+        <box size="0.15 0.15 0.2"/>  <!-- Must match visual -->
       </geometry>
     </collision>
@@ -37,5 +37,5 @@
     <parent link="tool0"/>
     <child link="simple_ee_link"/>
-    <origin xyz="0 -0.02 0.16" rpy="0 0 0"/>  <!-- 1cm offset from tool0 -->
+    <origin xyz="0 -0.02 0.11" rpy="0 0 0"/>  <!-- 1cm offset from tool0 -->
   </joint>
   <link name="camera_link"> </link>

Commit message: tmp save

File: src/end_effector_description/urdf/end_effector_withDriverSupport.xacro (robot description, xacro)
@@ -9,33 +9,14 @@
   <xacro:arg name="ur_type" default="ur10"/>
   <xacro:include filename="$(find ur_description)/urdf/ur.urdf.xacro"/>
- <!-- Simple rectangular end-effector -->
-  <link name="simple_ee_link">
-    <visual>
-      <geometry>
-        <box size="0.15 0.15 0.2"/>  <!-- Length, Width, Height -->
-      </geometry>
-      <material name="orange">
-        <color rgba="1.0 0.5 0.0 1.0"/>
-      </material>
-    </visual>
-    <collision>
-      <geometry>
-        <box size="0.15 0.15 0.2"/>  <!-- Must match visual -->
-      </geometry>
-    </collision>
-    <inertial>
-    <mass value="2.0"/>  <!-- 2kg mass -->
-    <!-- Calculated inertia for a rectangular prism -->
-    <inertia
-      ixx="0.01625" ixy="0.0" ixz="0.0"
-      iyy="0.0085" iyz="0.0"
-      izz="0.00425"/>
-  </inertial>
-  </link>
-  <!-- Fixed joint attaching to tool0 -->
-  <joint name="simple_ee_joint" type="fixed">
+  <xacro:include filename="$(find end_effector_description)/urdf/end_effector.urdf.xacro" />
+  <!-- This is the abstract link which the base of the claw attaches to. -->
+  <link name="end_effector_root_link"/>
+  <!-- Instantiate the claw by using its macro. -->
+  <xacro:end_effector prefix="" parent="end_effector_root_link" >
+  </xacro:end_effector>
+  <!-- Coupler between arm and end effector -->
+  <joint name="end_effector_coupler_joint" type="fixed">
     <parent link="tool0"/>
-    <child link="simple_ee_link"/>
-    <origin xyz="0 -0.02 0.11" rpy="0 0 0"/>  <!-- 1cm offset from tool0 -->
+    <child link="end_effector_root_link"/>
   </joint>
   <link name="camera_link"> </link>

Commit message: save progress

File: src/end_effector_description/urdf/end_effector_withDriverSupport.xacro (robot description, xacro)
@@ -2,6 +2,4 @@
 <!-- displays the end-effector with UR5e(no Moveit support)-->
 <robot name="end_effector_withDriverSupport" xmlns:xacro="http://ros.org/wiki/xacro">
-  <!-- Including the claw.urdf.xacro file to give scope to xacro:claw. Inclusion is a simple copy-and-paste of code. -->
-  <xacro:include filename="$(find end_effector_description)/urdf/end_effector.urdf.xacro" />
   <!-- UR5e robot arm -->
   <!-- URDF won't build if following args aren't defined. -->
@@ -9,14 +7,33 @@
   <xacro:arg name="ur_type" default="ur10"/>
   <xacro:include filename="$(find ur_description)/urdf/ur.urdf.xacro"/>
-  <xacro:include filename="$(find end_effector_description)/urdf/end_effector.urdf.xacro" />
-  <!-- This is the abstract link which the base of the claw attaches to. -->
-  <link name="end_effector_root_link"/>
-  <!-- Instantiate the claw by using its macro. -->
-  <xacro:end_effector prefix="" parent="end_effector_root_link" >
-  </xacro:end_effector>
-  <!-- Coupler between arm and end effector -->
-  <joint name="end_effector_coupler_joint" type="fixed">
+ <!-- Simple rectangular end-effector -->
+  <link name="simple_ee_link">
+    <visual>
+      <geometry>
+        <box size="0.15 0.15 0.2"/>  <!-- Length, Width, Height -->
+      </geometry>
+      <material name="orange">
+        <color rgba="1.0 0.5 0.0 1.0"/>
+      </material>
+    </visual>
+    <collision>
+      <geometry>
+        <box size="0.15 0.15 0.2"/>  <!-- Must match visual -->
+      </geometry>
+    </collision>
+    <inertial>
+    <mass value="2.0"/>  <!-- 2kg mass -->
+    <!-- Calculated inertia for a rectangular prism -->
+    <inertia
+      ixx="0.01625" ixy="0.0" ixz="0.0"
+      iyy="0.0085" iyz="0.0"
+      izz="0.00425"/>
+  </inertial>
+  </link>
+  <!-- Fixed joint attaching to tool0 -->
+  <joint name="simple_ee_joint" type="fixed">
     <parent link="tool0"/>
-    <child link="end_effector_root_link"/>
+    <child link="simple_ee_link"/>
+    <origin xyz="0 -0.02 0.11" rpy="0 0 0"/>  <!-- 1cm offset from tool0 -->
   </joint>
   <link name="camera_link"> </link>
